File: surge_protection.kicad_sch (KiCad schematic)
At the start: 21 parts, among them Q1 STP110N10F7, Q2 STP110N10F7, Q3 AON6284A, U3 NE555DR

Commit message: Add files via upload
Parts:
- removed R10, R4: R_1.1K_0603_1%, Resistor_SMD:R_0603_1608Metric, symbol JLCPartNumberLibrary:R_1.1K_0603
- added R20, R21: R_4.3K_0603_1%, Resistor_SMD:R_0603_1608Metric, symbol JLCPartNumberLibrary:R_4.3K_0603
Connections:
- net ADC1_IN3: now also R21.1
- net ADC1_IN4: now also R20.1
- net GND: now also R20.2, R21.2
Changed lines of the file:
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@@
+	)
+	(symbol
+		(lib_id "JLCPartNumberLibrary:R_4.3K_0603")
+		(at 220.98 90.17 0)
+		(unit 1)
+		(exclude_from_sim no)
+		(in_bom yes)
+		(on_board yes)
+		(dnp no)
+		(fields_autoplaced yes)
+		(property "Reference" "R21"
+			(at 223.52 88.8999 0)
+			(effects
+				(font
+					(size 1.27 1.27)
+				)
+				(justify left)
+			)
+		)
+		(property "Value" "R_4.3K_0603_1%"
+			(at 223.52 91.4399 0)
+			(effects
+				(font
+					(size 1.27 1.27)
+				)
+				(justify left)
+			)
+		)
+		(property "Footprint" "Resistor_SMD:R_0603_1608Metric"
+			(at 219.202 90.17 90)
+			(effects
+				(font
+					(size 1.27 1.27)
+				)
+				(hide yes)
+			)
+		)
+		(property "Datasheet" "~"
+			(at 220.98 90.17 0)
+			(effects
+				(font
+					(size 1.27 1.27)
+				)
+				(hide yes)
+			)
+		)
+		(property "Description" "Resistor"
+			(at 220.98 90.17 0)
+			(effects
+				(font
+					(size 1.27 1.27)
+				)
+				(hide yes)
+			)
+		)
+		(property "LCSC PN" "C2930099"
+			(at 220.98 90.17 0)
+			(effects
+				(font
+					(size 1.27 1.27)
+				)
+				(hide yes)
+			)
+		)
+		(pin "1"
+		)
+		(pin "2"
+		)
+		(instances
+			(project "EV_Design_Challenge"
+				(path "/24eb2c32-a4ca-4193-b269-5ddda1e66cf1/e43e326c-ccd5-43dc-9970-94ae69b64a29"
+					(reference "R21")
+					(unit 1)
+				)
+			)
+		)
 	)
 	(symbol
@@
 				(path "/24eb2c32-a4ca-4193-b269-5ddda1e66cf1/e43e326c-ccd5-43dc-9970-94ae69b64a29"
 					(reference "D3")
-					(unit 1)
-				)
-			)
-		)
-	)
-	(symbol
-		(lib_id "JLCPartNumberLibrary:R_1.1K_0603")
-		(at 220.98 90.17 0)
-		(unit 1)
-		(exclude_from_sim no)
-		(in_bom yes)
-		(on_board yes)
-		(dnp no)
-		(fields_autoplaced yes)
-		(property "Reference" "R4"
-			(at 223.52 88.8999 0)
-			(effects
-				(font
-					(size 1.27 1.27)
-				)
-				(justify left)
-			)
-		)
-		(property "Value" "R_1.1K_0603_1%"
-			(at 223.52 91.4399 0)
-			(effects
-				(font
-					(size 1.27 1.27)
-				)
-				(justify left)
-			)
-		)
-		(property "Footprint" "Resistor_SMD:R_0603_1608Metric"
-			(at 219.202 90.17 90)
-			(effects
-				(font
-					(size 1.27 1.27)
-				)
-				(hide yes)
-			)
-		)
-		(property "Datasheet" "~"
-			(at 220.98 90.17 0)
-			(effects
-				(font
-					(size 1.27 1.27)
-				)
-				(hide yes)
-			)
-		)
-		(property "Description" "Resistor"
-			(at 220.98 90.17 0)
-			(effects
-				(font
-					(size 1.27 1.27)
-				)
-				(hide yes)
-			)
-		)
-		(property "LCSC PN" "C22764"
-			(at 220.98 90.17 0)
-			(effects
-				(font
-					(size 1.27 1.27)
-				)
-				(hide yes)
-			)
-		)
-		(pin "1"
-		)
-		(pin "2"
-		)
-		(instances
-			(project "EV_Design_Challenge"
-				(path "/24eb2c32-a4ca-4193-b269-5ddda1e66cf1/e43e326c-ccd5-43dc-9970-94ae69b64a29"
-					(reference "R4")
 					(unit 1)
 				)
@@
 	)
 	(symbol
-		(lib_id "JLCPartNumberLibrary:R_1.1K_0603")
+		(lib_id "power:GND")
+		(at 148.59 99.06 0)
+		(unit 1)
+		(exclude_from_sim no)
+		(in_bom yes)
+		(on_board yes)
+		(dnp no)
+		(fields_autoplaced yes)
+		(property "Reference" "#PWR07"
+			(at 148.59 105.41 0)
+			(effects
+				(font
+					(size 1.27 1.27)
+				)
+				(hide yes)
+			)
+		)
+		(property "Value" "GND"
+			(at 148.59 104.14 0)
+			(effects
+				(font
+					(size 1.27 1.27)
+				)
+			)
+		)
+		(property "Footprint" ""
+			(at 148.59 99.06 0)
+			(effects
+				(font
+					(size 1.27 1.27)
+				)
+				(hide yes)
+			)
+		)
+		(property "Datasheet" ""
+			(at 148.59 99.06 0)
+			(effects
+				(font
+					(size 1.27 1.27)
+				)
+				(hide yes)
+			)
+		)
+		(property "Description" "Power symbol creates a global label with name \"GND\" , ground"
+			(at 148.59 99.06 0)
+			(effects
+				(font
+					(size 1.27 1.27)
+				)
+				(hide yes)
+			)
+		)
+		(pin "1"
+		)
+		(instances
+			(project "EV_Design_Challenge"
+				(path "/24eb2c32-a4ca-4193-b269-5ddda1e66cf1/e43e326c-ccd5-43dc-9970-94ae69b64a29"
+					(reference "#PWR07")
+					(unit 1)
+				)
+			)
+		)
+	)
+	(symbol
+		(lib_id "JLCPartNumberLibrary:R_4.3K_0603")
 		(at 193.04 90.17 0)
 		(unit 1)
@@
 		(dnp no)
 		(fields_autoplaced yes)
-		(property "Reference" "R10"
+		(property "Reference" "R20"
 			(at 195.58 88.8999 0)
 			(effects
@@
 			)
 		)
-		(property "Value" "R_1.1K_0603_1%"
+		(property "Value" "R_4.3K_0603_1%"
 			(at 195.58 91.4399 0)
 			(effects
@@
 			)
 		)
-		(property "LCSC PN" "C22764"
+		(property "LCSC PN" "C2930099"
 			(at 193.04 90.17 0)
 			(effects
@@
 			(project "EV_Design_Challenge"
 				(path "/24eb2c32-a4ca-4193-b269-5ddda1e66cf1/e43e326c-ccd5-43dc-9970-94ae69b64a29"
-					(reference "R10")
-					(unit 1)
-				)
-			)
-		)
-	)
-	(symbol
-		(lib_id "power:GND")
-		(at 148.59 99.06 0)
-		(unit 1)
-		(exclude_from_sim no)
-		(in_bom yes)
-		(on_board yes)
-		(dnp no)
-		(fields_autoplaced yes)
-		(property "Reference" "#PWR07"
-			(at 148.59 105.41 0)
-			(effects
-				(font
-					(size 1.27 1.27)
-				)
-				(hide yes)
-			)
-		)
-		(property "Value" "GND"
-			(at 148.59 104.14 0)
-			(effects
-				(font
-					(size 1.27 1.27)
-				)
-			)
-		)
-		(property "Footprint" ""
-			(at 148.59 99.06 0)
-			(effects
-				(font
-					(size 1.27 1.27)
-				)
-				(hide yes)
-			)
-		)
-		(property "Datasheet" ""
-			(at 148.59 99.06 0)
-			(effects
-				(font
-					(size 1.27 1.27)
-				)
-				(hide yes)
-			)
-		)
-		(property "Description" "Power symbol creates a global label with name \"GND\" , ground"
-			(at 148.59 99.06 0)
-			(effects
-				(font
-					(size 1.27 1.27)
-				)
-				(hide yes)
-			)
-		)
-		(pin "1"
-		)
-		(instances
-			(project "EV_Design_Challenge"
-				(path "/24eb2c32-a4ca-4193-b269-5ddda1e66cf1/e43e326c-ccd5-43dc-9970-94ae69b64a29"
-					(reference "#PWR07")
-					(unit 1)
-				)
+					(reference "R20")
+					(unit 1)
+				)
