File: EV_Design_Challenge.kicad_pcb (KiCad board)
At the start: 2 copper layers, 72 x 67 mm, 78 parts, among them J1 WAGO-2604-1102, J2 WAGO-2604-1102, J3 01x02_2.54mm_Header_Pins, J4 01x05_2.54mm_Header_Pins, J5 WAGO-2604-1102, Q1 STP110N10F7, Q2 STP110N10F7, Q3 AON6284A, SW1 SMT_Debug_Push_Button, U1 STM32G473CEUx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

Commit message: Add files via upload
Other:
- board text added: "5V STAT"
- board text added: "VOUT STAT"
Changed lines of the file:
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@@
 			(at 0 -1.43 0)
 			(layer "F.SilkS")
+			(hide yes)
 			(effects
 				(font
@@
 			(at 0 -1.43 0)
 			(layer "F.SilkS")
+			(hide yes)
 			(effects
 				(font
@@
 			(at 0 -1.17 0)
 			(layer "F.SilkS")
+			(hide yes)
 			(effects
 				(font
@@
 		(layer "F.SilkS" knockout)
 		(effects
+			(font
+				(size 0.6 0.6)
+				(thickness 0.12)
+				(bold yes)
+			)
+			(justify left bottom)
+		)
+	)
+	(gr_text "VOUT STAT"
+		(at 107 55 0)
+		(layer "F.SilkS" knockout)
+		(effects
+			(font
+				(size 0.6 0.6)
+				(thickness 0.12)
+				(bold yes)
+			)
+			(justify left bottom)
+		)
+	)
+	(gr_text "5V STAT"
+		(at 115.5 88 0)
+		(layer "F.SilkS" knockout)
+		(effects

Commit message: Add files via upload
Routing:
- net ADC1_IN4: track 69.3 -> 70.7 mm
Changed lines of the file:
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@@
 	)
 	(segment
-		(start 82.5 59.434315)
-		(end 82.5 73.5)
+		(start 82.5 73.5)
+		(end 82 74)
 		(width 0.2)
 		(layer "F.Cu")
@@
 	)
 	(segment
-		(start 93 56.5)
-		(end 85.434315 56.5)
+		(start 94 55.5)
+		(end 84 55.5)
 		(width 0.2)
 		(layer "F.Cu")
@@
 	)
 	(segment
-		(start 85.434315 56.5)
-		(end 82.5 59.434315)
+		(start 97 52.5)
+		(end 94 55.5)
 		(width 0.2)
 		(layer "F.Cu")
@@
 	)
 	(segment
-		(start 98.5 45.175)
-		(end 97 46.675)
-		(width 0.2)
-		(layer "F.Cu")
-		(net 27)
-	)
-	(segment
-		(start 97 52.5)
-		(end 93 56.5)
-		(width 0.2)
-		(layer "F.Cu")
-		(net 27)
-	)
-	(segment
 		(start 97 46.675)
 		(end 97 52.5)
-		(width 0.2)
-		(layer "F.Cu")
-		(net 27)
-	)
-	(segment
-		(start 82.5 73.5)
-		(end 82 74)
 		(width 0.2)
 		(layer "F.Cu")
@@
 		(width 0.2)
 		(layer "F.Cu")
+		(net 27)
+	)
+	(segment
+		(start 98.5 45.175)
+		(end 97 46.675)
+		(width 0.2)
+		(layer "F.Cu")
+		(net 27)
+	)
+	(segment
+		(start 84 55.5)
+		(end 82.5 57)
+		(width 0.2)
+		(layer "F.Cu")
+		(net 27)
+	)
+	(segment
+		(start 82.5 57)
+		(end 82.5 73.5)
+		(width 0.2)
+		(layer "F.Cu")
